File: V2.0/A2RAM128.v2.0.kicad_pcb (KiCad board)
At the start: 2 copper layers, 65.5 x 38.6 mm, 69 parts, among them U1 DIP-32_W15.24mm_Socket, U2 DIP-24_W7.62mm_Socket

Commit message: Add files via upload
Other:
- board text added: "128kB Bank Switched RAM card. Hardware design by Ralle Palaveev (c) 2025."
- board text removed: "128kB Bank Switched RAM card. Hardware design by Ralle Palaveev (c) 2024. For A2 computers with less than 64kB RAM."
Changed lines of the file:
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@@
 		)
 	)
-	(gr_text "128kB Bank Switched RAM card.\nHardware design by Ralle Palaveev (c) 2024.\nFor A2 computers with less than 64kB RAM."
+	(gr_text "128kB Bank Switched RAM card.\nHardware design by Ralle Palaveev (c) 2025.\n"
 		(at 133.223 111.633 0)
 		(layer "B.SilkS")

Commit message: Add files via upload
Other:
- board text added: "A2RAM128.v2.0 for Apple ][, (c) 2025 by Ralle Palaveev, https://apple2.co.uk/"
- board text removed: "A2RAM128.v2.0 for Apple ][, (c) 2024 by Ralle Palaveev, https://apple2.co.uk/"
Changed lines of the file:
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@@
 		)
 	)
-	(gr_text "A2RAM128.v2.0 for Apple ][, (c) 2024 by Ralle Palaveev, https://apple2.co.uk/"
+	(gr_text "A2RAM128.v2.0 for Apple ][, (c) 2025 by Ralle Palaveev, https://apple2.co.uk/"
 		(at 133.858 122.301 0)
 		(layer "F.SilkS")

Commit message: Add files via upload
Routing:
- net GND: track 63.3 -> 72.1 mm
Changed lines of the file:
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@@
+	)
+	(segment
+		(start 120.65 105.1814)
+		(end 120.65 100.457)
+		(width 0.25)
+		(layer "F.Cu")
+		(net 1)
+	)
+	(segment
+		(start 119.385 106.4464)
+		(end 120.65 105.1814)
+		(width 0.25)
+		(layer "F.Cu")
+		(net 1)
 	)
 	(segment
@@
 	)
 	(segment
+		(start 120.65 100.457)
+		(end 120.269 100.076)
+		(width 0.25)
+		(layer "F.Cu")
+		(net 1)
+	)
+	(segment
 		(start 127 119.38)
 		(end 127 117.856)
@@
 	)
 	(segment
-		(start 160.782 109.22)
-		(end 160.782 110.871)
+		(start 119.385 107.965)
+		(end 119.385 106.4464)
 		(width 0.25)
 		(layer "F.Cu")
@@
 		(net 1)
 	)
+	(segment
+		(start 160.782 109.22)
+		(end 160.782 111.1758)
+		(width 0.25)
+		(layer "F.Cu")
+		(net 1)
+	)
 	(via
 		(at 154.813 104.14)
@@
 	)
 	(via
-		(at 160.782 111.76)
+		(at 160.8074 112.1156)
 		(size 0.8)
 		(drill 0.4)
@@
 	)
 	(via
-		(at 160.782 110.871)
+		(at 160.782 111.1758)
 		(size 0.8)
 		(drill 0.4)
@@
 		(layers "F.Cu" "B.Cu")
 		(free yes)
-		(net 1)
-	)
-	(segment
-		(start 161.544 111.76)
-		(end 163.83 114.046)
-		(width 0.25)
-		(layer "B.Cu")
 		(net 1)
 	)
@@
 	)
 	(segment
+		(start 160.782 112.0902)
+		(end 160.8074 112.1156)
+		(width 0.25)
+		(layer "B.Cu")
+		(net 1)
+	)
+	(segment
 		(start 104.013 122.5804)
 		(end 104.013 123.825)
@@
 	)
 	(segment
-		(start 160.782 111.76)
-		(end 161.544 111.76)
-		(width 0.25)
-		(layer "B.Cu")
-		(net 1)
-	)
-	(segment
-		(start 160.782 110.871)
-		(end 160.782 111.76)
+		(start 161.8996 112.1156)
+		(end 163.83 114.046)
 		(width 0.25)
 		(layer "B.Cu")
@@
 		(start 125.5268 122.2756)
 		(end 104.3178 122.2756)
+		(width 0.25)
+		(layer "B.Cu")
+		(net 1)
+	)
+	(segment
+		(start 160.782 111.1758)
+		(end 160.782 112.0902)
 		(width 0.25)
 		(layer "B.Cu")
@@
 	)
 	(segment
+		(start 160.8074 112.1156)
+		(end 161.8996 112.1156)
+		(width 0.25)
+		(layer "B.Cu")
+		(net 1)
+	)
+	(segment
+		(start 160.881 114.046)
+		(end 163.83 114.046)
+		(width 1.5)
+		(layer "F.Cu")
+		(net 2)
+	)
+	(segment
 		(start 155.956 114.173)
 		(end 155.956 115.824)
@@
 	)
 	(segment
+		(start 160.754 114.173)
+		(end 160.881 114.046)
+		(width 0.8)
+		(layer "F.Cu")
+		(net 2)
+	)
+	(segment
 		(start 147.325 119.375)
 		(end 147.32 119.38)
@@
 	)
 	(segment
-		(start 163.703 114.173)
-		(end 163.83 114.046)
+		(start 155.956 114.173)
+		(end 160.754 114.173)
 		(width 0.8)
 		(layer "F.Cu")
@@
 		(layer "F.Cu")
 		(net 2)
-	)
-	(segment
-		(start 155.956 114.173)
-		(end 163.703 114.173)
-		(width 0.8)
-		(layer "F.Cu")
-		(net 2)
